Commit message: Started xacro model

File: raider_3197_description/urdf/raider_3197.xacro (robot description, xacro)
@@ -1,7 +1,8 @@
 <?xml version="1.0"?>
-<robot name="mantis_uav" xmlns:xacro="http://ros.org/wiki/xacro">
+<robot name="raider_3197" xmlns:xacro="http://ros.org/wiki/xacro">
 	<!-- Constants -->
 	<xacro:property name="pi" value="3.1415926535897931"/>
 	<!-- Import macros -->
+	<!--
 	<xacro:include filename="$(find mantis_description)/urdf/visual_servo.xacro" />
 	<xacro:include filename="$(find mantis_description)/urdf/frame_battery.xacro" />
@@ -13,8 +14,13 @@
 	<xacro:include filename="$(find mantis_description)/urdf/arm_link.xacro" />
 	<xacro:include filename="$(find mantis_description)/urdf/motor_joint.xacro" />
+	-->
+	<xacro:include filename="$(find raider_3197_description)/urdf/wheel_front_joint.xacro" />
+	<xacro:include filename="$(find raider_3197_description)/urdf/wheel_front_link.xacro" />
+	<xacro:include filename="$(find raider_3197_description)/urdf/wheel_rear_joint.xacro" />
+	<xacro:include filename="$(find raider_3197_description)/urdf/wheel_rear_link.xacro" />
 	<!-- Import all Gazebo-customization elements, including Gazebo colors -->
-	<xacro:include filename="$(find mantis_description)/urdf/mantis.gazebo" />
+	<xacro:include filename="$(find raider_3197_description)/urdf/raider_3197.gazebo" />
 	<!-- Import Rviz colors -->
-	<xacro:include filename="$(find mantis_description)/urdf/materials.xacro" />
+	<xacro:include filename="$(find raider_3197_description)/urdf/materials.xacro" />
 	<!-- Used for fixing robot to Gazebo 'base_link' -->
 	<link name="world"/>
@@ -26,18 +32,19 @@
 	<link name="base_link">
 		<inertial>
-			<mass value="1.80497" />
-			<inertia ixx="0.02961" iyy="0.02933" izz="0.05342" ixy="0.0" ixz="0.00004" iyz="0.0" />
+			<mass value="1.0" />
+			<inertia ixx="0.004167" iyy="0.011042" izz="0.01354" ixy="0.0" ixz="0.0" iyz="0.0" />
 		</inertial>
 		<collision name='collision_base_link'>
 			<geometry>
-				<cylinder radius="0.105" length="0.03"/>
+				<box size="0.350 0.200 0.075"/>
 			</geometry>
 		</collision>
 		<visual name='visual_base_link'>
 			<geometry>
-				<cylinder radius="0.105" length="0.03"/>
+				<box size="0.350 0.200 0.075"/>
 			</geometry>
 			<material name="orange"/>
 		</visual>
+		<!--
 		<xacro:frame_battery suffix="battery_primary" size="0.052 0.146 0.034" color="blue" xyz="0.0 0.0 0.032" rpy="0.0 0.0 0.0" />
 		<xacro:frame_servo suffix="servo_shoulder" size="0.0285 0.034 0.0465" color="black" xyz="0.01425 0.019 -0.015" rpy="${-pi/2} 0 ${pi}" />
@@ -60,7 +67,15 @@
 		<xacro:frame_skid suffix="skid_5" length="0.12" radius="0.008" color="white" xyz="0.2382 -0.1375 -0.075" rpy="0 0 0" />
 		<xacro:frame_skid suffix="skid_6" length="0.12" radius="0.008" color="white" xyz="-0.2382 0.1375 -0.075" rpy="0 0 0" />
+		-->
 	</link>
-	<xacro:arm_joint suffix="shoulder" parent="base_link" child="link_upperarm" xyz="0 0 -0.05025" rpy="${pi/2} ${pi/2} 0" />
-	<xacro:arm_link suffix="upperarm" />
+	<xacro:wheel_front_joint suffix="wheel_front_left" parent="base_link" xyz="0.175 0.11 -0.05" rpy="${pi/2} ${pi/2} 0" />
+	<xacro:wheel_front_link suffix="wheel_front_left" />
+	<xacro:wheel_front_joint suffix="wheel_front_right" parent="base_link" xyz="0.175 -0.11 -0.05" rpy="${pi/2} ${pi/2} 0" />
+	<xacro:wheel_front_link suffix="wheel_front_right" />
+	<xacro:wheel_rear_joint suffix="wheel_rear_left" parent="base_link" xyz="-0.175 0.12 -0.0375" rpy="${pi/2} ${pi/2} 0" />
+	<xacro:wheel_rear_link suffix="wheel_rear_left" />
+	<xacro:wheel_rear_joint suffix="wheel_rear_right" parent="base_link" xyz="-0.175 -0.12 -0.0375" rpy="${pi/2} ${pi/2} 0" />
+	<xacro:wheel_rear_link suffix="wheel_rear_right" />
+	<!--
 	<xacro:arm_joint suffix="elbow" parent="link_upperarm" child="link_forearm" xyz="0.18325 0 0" rpy="0 0 0" />
 	<xacro:arm_link suffix="forearm" />
@@ -71,3 +86,4 @@
 	<xacro:motor_joint motor_number="5" parent="base_link" xyz="0.2382 -0.1375 0.0455" direction="ccw" />
 	<xacro:motor_joint motor_number="6" parent="base_link" xyz="-0.2382 0.1375 0.0455" direction="cw" />
+	-->
 </robot>

Commit message: Suspension!

File: raider_3197_description/urdf/raider_3197.xacro (robot description, xacro)
@@ -4,15 +4,4 @@
 	<xacro:property name="pi" value="3.1415926535897931"/>
 	<!-- Import macros -->
-	<!--
-	<xacro:include filename="$(find mantis_description)/urdf/visual_servo.xacro" />
-	<xacro:include filename="$(find mantis_description)/urdf/frame_battery.xacro" />
-	<xacro:include filename="$(find mantis_description)/urdf/frame_servo.xacro" />
-	<xacro:include filename="$(find mantis_description)/urdf/frame_arm.xacro" />
-	<xacro:include filename="$(find mantis_description)/urdf/frame_motor.xacro" />
-	<xacro:include filename="$(find mantis_description)/urdf/frame_skid.xacro" />
-	<xacro:include filename="$(find mantis_description)/urdf/arm_joint.xacro" />
-	<xacro:include filename="$(find mantis_description)/urdf/arm_link.xacro" />
-	<xacro:include filename="$(find mantis_description)/urdf/motor_joint.xacro" />
-	-->
 	<xacro:include filename="$(find raider_3197_description)/urdf/wheel_front_joint.xacro" />
 	<xacro:include filename="$(find raider_3197_description)/urdf/wheel_front_link.xacro" />
@@ -46,30 +35,8 @@
 			<material name="orange"/>
 		</visual>
-		<!--
-		<xacro:frame_battery suffix="battery_primary" size="0.052 0.146 0.034" color="blue" xyz="0.0 0.0 0.032" rpy="0.0 0.0 0.0" />
-		<xacro:frame_servo suffix="servo_shoulder" size="0.0285 0.034 0.0465" color="black" xyz="0.01425 0.019 -0.015" rpy="${-pi/2} 0 ${pi}" />
-		<xacro:frame_arm suffix="arm_1" length="0.17" radius="0.015" color="white" xyz="0 -0.19 0" rpy="${pi/2} 0 0" />
-		<xacro:frame_arm suffix="arm_2" length="0.17" radius="0.015" color="white" xyz="0 0.19 0" rpy="${pi/2} 0 0" />
-		<xacro:frame_arm suffix="arm_3" length="0.17" radius="0.015" color="red" xyz="0.165 0.095 0" rpy="${pi/2} 0 ${2*pi/3}" />
-		<xacro:frame_arm suffix="arm_4" length="0.17" radius="0.015" color="white" xyz="-0.165 -0.095 0" rpy="${pi/2} 0 ${2*pi/3}" />
-		<xacro:frame_arm suffix="arm_5" length="0.17" radius="0.015" color="red" xyz="0.165 -0.095 0" rpy="${pi/2} 0 ${pi/3}" />
-		<xacro:frame_arm suffix="arm_6" length="0.17" radius="0.015" color="white" xyz="-0.165 0.095 0" rpy="${pi/2} 0 ${pi/3}" />
-		<xacro:frame_motor suffix="motor_1" length="0.024" radius="0.014" color="grey" xyz="0 -0.275 0.027" rpy="0 0 0" />
-		<xacro:frame_motor suffix="motor_2" length="0.024" radius="0.014" color="grey" xyz="0 0.275 0.027" rpy="0 0 0" />
-		<xacro:frame_motor suffix="motor_3" length="0.024" radius="0.014" color="grey" xyz="0.2382 0.1375 0.027" rpy="0 0 0" />
-		<xacro:frame_motor suffix="motor_4" length="0.024" radius="0.014" color="grey" xyz="-0.2382 -0.1375 0.027" rpy="0 0 0" />
-		<xacro:frame_motor suffix="motor_5" length="0.024" radius="0.014" color="grey" xyz="0.2382 -0.1375 0.027" rpy="0 0 0" />
-		<xacro:frame_motor suffix="motor_6" length="0.024" radius="0.014" color="grey" xyz="-0.2382 0.1375 0.027" rpy="0 0 0" />
-		<xacro:frame_skid suffix="skid_1" length="0.12" radius="0.008" color="white" xyz="0 -0.275 -0.075" rpy="0 0 0" />
-		<xacro:frame_skid suffix="skid_2" length="0.12" radius="0.008" color="white" xyz="0 0.275 -0.075" rpy="0 0 0" />
-		<xacro:frame_skid suffix="skid_3" length="0.12" radius="0.008" color="white" xyz="0.2382 0.1375 -0.075" rpy="0 0 0" />
-		<xacro:frame_skid suffix="skid_4" length="0.12" radius="0.008" color="white" xyz="-0.2382 -0.1375 -0.075" rpy="0 0 0" />
-		<xacro:frame_skid suffix="skid_5" length="0.12" radius="0.008" color="white" xyz="0.2382 -0.1375 -0.075" rpy="0 0 0" />
-		<xacro:frame_skid suffix="skid_6" length="0.12" radius="0.008" color="white" xyz="-0.2382 0.1375 -0.075" rpy="0 0 0" />
-		-->
 	</link>
-	<xacro:wheel_front_joint suffix="wheel_front_left" parent="base_link" xyz="0.175 0.11 -0.05" rpy="${pi/2} ${pi/2} 0" />
+	<xacro:wheel_front_joint suffix="wheel_front_left" parent="base_link" xyz="0.175 0.11 -0.0375" rpy="${pi/2} ${pi/2} 0" />
 	<xacro:wheel_front_link suffix="wheel_front_left" />
-	<xacro:wheel_front_joint suffix="wheel_front_right" parent="base_link" xyz="0.175 -0.11 -0.05" rpy="${pi/2} ${pi/2} 0" />
+	<xacro:wheel_front_joint suffix="wheel_front_right" parent="base_link" xyz="0.175 -0.11 -0.0375" rpy="${pi/2} ${pi/2} 0" />
 	<xacro:wheel_front_link suffix="wheel_front_right" />
 	<xacro:wheel_rear_joint suffix="wheel_rear_left" parent="base_link" xyz="-0.175 0.12 -0.0375" rpy="${pi/2} ${pi/2} 0" />
@@ -77,13 +44,3 @@
 	<xacro:wheel_rear_joint suffix="wheel_rear_right" parent="base_link" xyz="-0.175 -0.12 -0.0375" rpy="${pi/2} ${pi/2} 0" />
 	<xacro:wheel_rear_link suffix="wheel_rear_right" />
-	<!--
-	<xacro:arm_joint suffix="elbow" parent="link_upperarm" child="link_forearm" xyz="0.18325 0 0" rpy="0 0 0" />
-	<xacro:arm_link suffix="forearm" />
-	<xacro:motor_joint motor_number="1" parent="base_link" xyz="0 -0.275 0.0455" direction="cw" />
-	<xacro:motor_joint motor_number="2" parent="base_link" xyz="0 0.275 0.0475" direction="ccw" />
-	<xacro:motor_joint motor_number="3" parent="base_link" xyz="0.2382 0.1375 0.0455" direction="cw" />
-	<xacro:motor_joint motor_number="4" parent="base_link" xyz="-0.2382 -0.1375 0.0455" direction="ccw" />
-	<xacro:motor_joint motor_number="5" parent="base_link" xyz="0.2382 -0.1375 0.0455" direction="ccw" />
-	<xacro:motor_joint motor_number="6" parent="base_link" xyz="-0.2382 0.1375 0.0455" direction="cw" />
-	-->
 </robot>

File: raider_3197_description/urdf/wheel_front_joint.xacro (robot description, xacro)
@@ -1,26 +1,15 @@
 <?xml version="1.0"?>
 <robot xmlns:xacro="http://ros.org/wiki/xacro">
+	<xacro:include filename="$(find raider_3197_description)/urdf/axle_joint.xacro" />
+	<xacro:include filename="$(find raider_3197_description)/urdf/suspension_joint.xacro" />
 	<xacro:macro name="wheel_front_joint" params="suffix parent xyz rpy">
-		<joint name="joint_${suffix}" type="continuous">
-			<parent link="${parent}"/>
-			<child link="link_${suffix}"/>
-			<origin xyz="${xyz}" rpy="${rpy}"/>
-			<axis xyz="0 0 1"/>
-			<limit effort="1000" velocity="1000"/>
-			<!--
-			<dynamics damping="0.1" friction="0.0"/>
-			-->
-		</joint>
-		<!--
-		<transmission name="trans_${suffix}">
-			<type>transmission_interface/SimpleTransmission</type>
-			<joint name="joint_${suffix}">
-				<hardwareInterface>hardware_interface/EffortJointInterface</hardwareInterface>
-			</joint>
-			<actuator name="motor_${suffix}">
-				<mechanicalReduction>1</mechanicalReduction>
-			</actuator>
-		</transmission>
-		-->
+		<xacro:suspension_joint suffix="${suffix}_axle" parent="${parent}" xyz="${xyz}" rpy="0 0 0" />
+		<link name="link_${suffix}_axle">
+			<inertial>
+				<mass value="0.025" />
+				<inertia ixx="5.8083e-4" ixy="0" ixz="0" iyy="3.0833e-5" iyz="0" izz="5.9083e-4" />
+			</inertial>
+		</link>
+		<xacro:axle_joint suffix="${suffix}" parent="link_${suffix}_axle" xyz="0 0 0" rpy="${rpy}" />
 	</xacro:macro>
 </robot>

File: raider_3197_description/urdf/wheel_rear_joint.xacro (robot description, xacro)
@@ -1,15 +1,15 @@
 <?xml version="1.0"?>
 <robot xmlns:xacro="http://ros.org/wiki/xacro">
+	<xacro:include filename="$(find raider_3197_description)/urdf/axle_joint.xacro" />
+	<xacro:include filename="$(find raider_3197_description)/urdf/suspension_joint.xacro" />
 	<xacro:macro name="wheel_rear_joint" params="suffix parent xyz rpy">
-		<joint name="joint_${suffix}" type="continuous">
-			<parent link="${parent}"/>
-			<child link="link_${suffix}"/>
-			<origin xyz="${xyz}" rpy="${rpy}"/>
-			<axis xyz="0 0 1"/>
-			<limit effort="1000" velocity="1000"/>
-			<!--
-			<dynamics damping="0.1" friction="0.0"/>
-			-->
-		</joint>
+		<xacro:suspension_joint suffix="${suffix}_axle" parent="${parent}" xyz="${xyz}" rpy="0 0 0" />
+		<link name="link_${suffix}_axle">
+			<inertial>
+				<mass value="0.025" />
+				<inertia ixx="5.8083e-4" ixy="0" ixz="0" iyy="3.0833e-5" iyz="0" izz="5.9083e-4" />
+			</inertial>
+		</link>
+		<xacro:axle_joint suffix="${suffix}" parent="link_${suffix}_axle" xyz="0 0 0" rpy="${rpy}" />
 		<transmission name="trans_${suffix}">
 			<type>transmission_interface/SimpleTransmission</type>

Commit message: Mesh is looking good

File: raider_3197_description/urdf/raider_3197.xacro (robot description, xacro)
@@ -26,21 +26,25 @@
 		<collision name='collision_base_link'>
 			<geometry>
-				<box size="0.350 0.200 0.075"/>
+				<box size="0.315 0.12 0.08"/>
 			</geometry>
 		</collision>
 		<visual name='visual_base_link'>
+			<origin xyz="0 0 -0.04" rpy="0 0 0"/>
 			<geometry>
+				<!--
 				<box size="0.350 0.200 0.075"/>
+				-->
+				<mesh filename="package://raider_3197_description/meshes/raider_3197_shell.stl" scale="0.01 0.01 0.01"/>
 			</geometry>
 			<material name="orange"/>
 		</visual>
 	</link>
-	<xacro:wheel_front_joint suffix="wheel_front_left" parent="base_link" xyz="0.175 0.11 -0.0375" rpy="${pi/2} ${pi/2} 0" />
+	<xacro:wheel_front_joint suffix="wheel_front_left" parent="base_link" xyz="0.1225 0.06 -0.0375" rpy="${pi/2} ${pi/2} 0" />
 	<xacro:wheel_front_link suffix="wheel_front_left" />
-	<xacro:wheel_front_joint suffix="wheel_front_right" parent="base_link" xyz="0.175 -0.11 -0.0375" rpy="${pi/2} ${pi/2} 0" />
+	<xacro:wheel_front_joint suffix="wheel_front_right" parent="base_link" xyz="0.1225 -0.06 -0.0375" rpy="${pi/2} ${pi/2} 0" />
 	<xacro:wheel_front_link suffix="wheel_front_right" />
-	<xacro:wheel_rear_joint suffix="wheel_rear_left" parent="base_link" xyz="-0.175 0.12 -0.0375" rpy="${pi/2} ${pi/2} 0" />
+	<xacro:wheel_rear_joint suffix="wheel_rear_left" parent="base_link" xyz="-0.1225 0.07 -0.0375" rpy="${pi/2} ${pi/2} 0" />
 	<xacro:wheel_rear_link suffix="wheel_rear_left" />
-	<xacro:wheel_rear_joint suffix="wheel_rear_right" parent="base_link" xyz="-0.175 -0.12 -0.0375" rpy="${pi/2} ${pi/2} 0" />
+	<xacro:wheel_rear_joint suffix="wheel_rear_right" parent="base_link" xyz="-0.1225 -0.07 -0.0375" rpy="${pi/2} ${pi/2} 0" />
 	<xacro:wheel_rear_link suffix="wheel_rear_right" />
 </robot>

File: raider_3197_description/urdf/wheel_front_link.xacro (robot description, xacro)
@@ -11,5 +11,5 @@
 				<origin xyz="0 0 0" rpy="0 0 0"/>
 				<geometry>
-					<cylinder radius="0.03" length="0.02"/>
+					<cylinder radius="0.03" length="0.015"/>
 				</geometry>
 			</collision>
@@ -17,5 +17,5 @@
 				<origin xyz="0 0 0" rpy="0 0 0"/>
 				<geometry>
-					<cylinder radius="0.03" length="0.02"/>
+					<cylinder radius="0.03" length="0.015"/>
 					<!--
 					<mesh filename="package://mantis_description/meshes/FR12-H101.stl" scale="0.001 0.001 0.001"/>

File: raider_3197_description/urdf/wheel_rear_link.xacro (robot description, xacro)
@@ -11,5 +11,5 @@
 				<origin xyz="0 0 0" rpy="0 0 0"/>
 				<geometry>
-					<cylinder radius="0.03" length="0.04"/>
+					<cylinder radius="0.03" length="0.03"/>
 				</geometry>
 			</collision>
@@ -17,5 +17,5 @@
 				<origin xyz="0 0 0" rpy="0 0 0"/>
 				<geometry>
-					<cylinder radius="0.03" length="0.04"/>
+					<cylinder radius="0.03" length="0.03"/>
 					<!--
 					<mesh filename="package://mantis_description/meshes/FR12-H101.stl" scale="0.001 0.001 0.001"/>
